Commit message: first commit

File: install/reto_m6/share/reto_m6/urdf/reto_robot.urdf (robot description, URDF)
Before this commit: robot reto_robot, 2 links, 1 joints
Links:
- link arm_link: geometry collision cylinder length=0.3 radius=0.05; visual cylinder length=0.3 radius=0.05
- link base_link: geometry collision box size=0.2 0.2 0.1; visual box size=0.2 0.2 0.1
Joints:
- joint base_to_arm: limit lower=-3.14 upper=3.14 effort=10.0 velocity=1.0 -> lower=-3.14 upper=3.14 effort=100 velocity=1.0
